File: hardware/fusion/WiFiPicoDMX_RevA.sch (EAGLE design)
At the start: 38 parts, among them J1 PANEL XLR-5: COM,-,+,SHELL, J2 PANEL DIN-5 MIDI IN, J3 FREE GPIO PADS, J4 ANALOG PADS, J5 RESERVED SIGNAL TEST PADS, J6 POWER/DMX TEST PADS, SW1 PTS810SJM250SMTR LFS RESET (N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, U1 Raspberry Pi Pico 2 W, U2 ISOW1412DFMR, U3 HCPL-0700-500E

Commit message: hardware: standardize resistors on 0402
Parts:
- R10, R11: value 0R 5% 0.1W 0603 Yageo RC0603JR-070RL CMC BYPASS FIT -> 0R 5% 0.063W 0402 Yageo RC0402JR-070RL CMC BYPASS FIT; device WiFiPicoDMX_RevA_embedded:RES0603 -> WiFiPicoDMX_RevA_embedded:RES0402
- R4, R5: value 220R 1% 0.1W 0603 Yageo RC0603FR-07220RL -> 220R 1% 0.063W 0402 Yageo RC0402FR-07220RL; device WiFiPicoDMX_RevA_embedded:RES0603 -> WiFiPicoDMX_RevA_embedded:RES0402
- R6: value 4.7k 1% 0.1W 0603 Yageo RC0603FR-074K7L -> 4.7k 1% 0.063W 0402 Yageo RC0402FR-074K7L; device WiFiPicoDMX_RevA_embedded:RES0603 -> WiFiPicoDMX_RevA_embedded:RES0402
- R7: value 47k 1% 0.1W 0603 Yageo RC0603FR-0747KL -> 47k 1% 0.063W 0402 Yageo RC0402FR-0747KL; device WiFiPicoDMX_RevA_embedded:RES0603 -> WiFiPicoDMX_RevA_embedded:RES0402
- R8, R9: value 1k 1% 0.1W 0603 Yageo RC0603FR-071KL -> 1k 1% 0.063W 0402 Yageo RC0402FR-071KL; device WiFiPicoDMX_RevA_embedded:RES0603 -> WiFiPicoDMX_RevA_embedded:RES0402
Changed lines of the file:
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@@
         <part name="F1" library="WiFiPicoDMX_RevA_embedded" deviceset="PPTC1206" device="" value="1206L050YR 0.5A HOLD"/>
         <part name="SW1" library="WiFiPicoDMX_RevA_embedded" deviceset="SWITCH_SMD" device="" value="PTS810SJM250SMTR LFS RESET (NO)"/>
-        <part name="R8" library="WiFiPicoDMX_RevA_embedded" deviceset="RES0603" device="" value="1k 1% 0.1W 0603 Yageo RC0603FR-071KL"/>
+        <part name="R8" library="WiFiPicoDMX_RevA_embedded" deviceset="RES0402" device="" value="1k 1% 0.063W 0402 Yageo RC0402FR-071KL"/>
         <part name="D3" library="WiFiPicoDMX_RevA_embedded" deviceset="LED0603" device="" value="PWR GREEN Lite-On LTST-C190KGKT"/>
-        <part name="R9" library="WiFiPicoDMX_RevA_embedded" deviceset="RES0603" device="" value="1k 1% 0.1W 0603 Yageo RC0603FR-071KL"/>
+        <part name="R9" library="WiFiPicoDMX_RevA_embedded" deviceset="RES0402" device="" value="1k 1% 0.063W 0402 Yageo RC0402FR-071KL"/>
         <part name="D4" library="WiFiPicoDMX_RevA_embedded" deviceset="LED0603" device="" value="DMX YELLOW Lite-On LTST-C190KSKT"/>
         <part name="J3" library="WiFiPicoDMX_RevA_embedded" deviceset="PADBANK17" device="" value="FREE GPIO PADS"/>
@@
         <part name="C9" library="WiFiPicoDMX_RevA_embedded" deviceset="CAP0603" device="" value="1uF 50V 10% X5R 0603 CL10A105KB8NNNC VISOOUT 2-4mm"/>
         <part name="L1" library="WiFiPicoDMX_RevA_embedded" deviceset="CMC_OPTION" device="" value="ACT45B-510-2P-TL003 - DNP"/>
-        <part name="R10" library="WiFiPicoDMX_RevA_embedded" deviceset="RES0603" device="" value="0R 5% 0.1W 0603 Yageo RC0603JR-070RL CMC BYPASS FIT"/>
-        <part name="R11" library="WiFiPicoDMX_RevA_embedded" deviceset="RES0603" device="" value="0R 5% 0.1W 0603 Yageo RC0603JR-070RL CMC BYPASS FIT"/>
+        <part name="R10" library="WiFiPicoDMX_RevA_embedded" deviceset="RES0402" device="" value="0R 5% 0.063W 0402 Yageo RC0402JR-070RL CMC BYPASS FIT"/>
+        <part name="R11" library="WiFiPicoDMX_RevA_embedded" deviceset="RES0402" device="" value="0R 5% 0.063W 0402 Yageo RC0402JR-070RL CMC BYPASS FIT"/>
         <part name="D1" library="WiFiPicoDMX_RevA_embedded" deviceset="SM712" device="" value="SM712.TCT"/>
         <part name="J1" library="WiFiPicoDMX_RevA_embedded" deviceset="PANEL_DMX4" device="" value="PANEL XLR-5: COM,-,+,SHELL"/>
         <part name="J2" library="WiFiPicoDMX_RevA_embedded" deviceset="PANEL_MIDI5" device="" value="PANEL DIN-5 MIDI IN"/>
-        <part name="R4" library="WiFiPicoDMX_RevA_embedded" deviceset="RES0603" device="" value="220R 1% 0.1W 0603 Yageo RC0603FR-07220RL"/>
-        <part name="R5" library="WiFiPicoDMX_RevA_embedded" deviceset="RES0603" device="" value="220R 1% 0.1W 0603 Yageo RC0603FR-07220RL"/>
+        <part name="R4" library="WiFiPicoDMX_RevA_embedded" deviceset="RES0402" device="" value="220R 1% 0.063W 0402 Yageo RC0402FR-07220RL"/>
+        <part name="R5" library="WiFiPicoDMX_RevA_embedded" deviceset="RES0402" device="" value="220R 1% 0.063W 0402 Yageo RC0402FR-07220RL"/>
         <part name="D2" library="WiFiPicoDMX_RevA_embedded" deviceset="DIODE_SOD323" device="" value="1N4148WS-E3-08"/>
         <part name="U3" library="WiFiPicoDMX_RevA_embedded" deviceset="HCPL_0700_500E" device="" value="HCPL-0700-500E"/>
-        <part name="R6" library="WiFiPicoDMX_RevA_embedded" deviceset="RES0603" device="" value="4.7k 1% 0.1W 0603 Yageo RC0603FR-074K7L"/>
-        <part name="R7" library="WiFiPicoDMX_RevA_embedded" deviceset="RES0603" device="" value="47k 1% 0.1W 0603 Yageo RC0603FR-0747KL"/>
+        <part name="R6" library="WiFiPicoDMX_RevA_embedded" deviceset="RES0402" device="" value="4.7k 1% 0.063W 0402 Yageo RC0402FR-074K7L"/>
+        <part name="R7" library="WiFiPicoDMX_RevA_embedded" deviceset="RES0402" device="" value="47k 1% 0.063W 0402 Yageo RC0402FR-0747KL"/>
         <part name="C7" library="WiFiPicoDMX_RevA_embedded" deviceset="CAP0402" device="" value="100nF 16V 10% X7R 0402 CL05B104KO5NNNC MIDI VCC"/>
       </parts>
