File: hardware/fusion/WiFiPicoDMX_RevA.brd (EAGLE design)
At the start: 95 x 100 mm, 37 parts, among them J1 JST XH B4B-XH-A DMX: COM,-,+,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, J2 JST XH B5B-XH-A MIDI: 1,2,3,4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, J3 FREE GPIO PADS, J4 ANALOG PADS, J5 RESERVED SIGNAL TEST PADS, SW1 PTS810SJM250SMTR LFS RESET (N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, U1 Raspberry Pi Pico 2 W, U2 ISOW1412DFMR, U3 HCPL-0700-500E

Commit message: hardware: link Fusion design to used component library
Parts:
- C1, C2, C4, C6, C7: device WiFiPicoDMX_RevA_embedded:CAPC1005X60 -> WiFiPicoDMX_RevA_used:CAPC1005X60
- C3, C5: device WiFiPicoDMX_RevA_embedded:CAPC2012X110 -> WiFiPicoDMX_RevA_used:CAPC2012X110
- C8, C9: device WiFiPicoDMX_RevA_embedded:CAPC1608X85 -> WiFiPicoDMX_RevA_used:CAPC1608X85
- D1: device WiFiPicoDMX_RevA_embedded:SOT23_ -> WiFiPicoDMX_RevA_used:SOT23_
- D2: device WiFiPicoDMX_RevA_embedded:SOD323_VISHAY -> WiFiPicoDMX_RevA_used:SOD323_VISHAY
- D3, D4: device WiFiPicoDMX_RevA_embedded:LEDC1608X55N_FLAT-B -> WiFiPicoDMX_RevA_used:LEDC1608X55N_FLAT-B
- F1: device WiFiPicoDMX_RevA_embedded:PPTC1206_1206L050YR -> WiFiPicoDMX_RevA_used:PPTC1206_1206L050YR
- FB1, FB2: device WiFiPicoDMX_RevA_embedded:INDC1006X60N -> WiFiPicoDMX_RevA_used:INDC1006X60N
- J1: device WiFiPicoDMX_RevA_embedded:B4B-XH-A -> WiFiPicoDMX_RevA_used:B4B-XH-A
- J2: device WiFiPicoDMX_RevA_embedded:B5B-XH-A -> WiFiPicoDMX_RevA_used:B5B-XH-A
- J3: device WiFiPicoDMX_RevA_embedded:PADBANK17 -> WiFiPicoDMX_RevA_used:PADBANK17
- J4: device WiFiPicoDMX_RevA_embedded:PADBANK5 -> WiFiPicoDMX_RevA_used:PADBANK5
- J5: device WiFiPicoDMX_RevA_embedded:PADBANK7 -> WiFiPicoDMX_RevA_used:PADBANK7
- L1: device WiFiPicoDMX_RevA_embedded:ACT45B_4P5X3P2 -> WiFiPicoDMX_RevA_used:ACT45B_4P5X3P2
- R1, R10, R11, R2, R3, R4, R5, R6, R7, R8, R9: device WiFiPicoDMX_RevA_embedded:RESC1005X40 -> WiFiPicoDMX_RevA_used:RESC1005X40
- SW1: device WiFiPicoDMX_RevA_embedded:PTS810_J_LEAD -> WiFiPicoDMX_RevA_used:PTS810_J_LEAD
- U1: device WiFiPicoDMX_RevA_embedded:PICO_2_W_DEVELOPMENT_BOARD -> WiFiPicoDMX_RevA_used:PICO_2_W_DEVELOPMENT_BOARD
- U2: device WiFiPicoDMX_RevA_embedded:DFM0020A_TI -> WiFiPicoDMX_RevA_used:DFM0020A_TI
- U3: device WiFiPicoDMX_RevA_embedded:HCPL0700_SO8 -> WiFiPicoDMX_RevA_used:HCPL0700_SO8
